File: Hardware/pcb/ZigerBot/ZigerBot.kicad_pcb (KiCad board)
At the start: 2 copper layers, 105 parts, among them J1 Motor A, J10 ICSP, J2 M Power, J3 Motor B, J4 4 Pin Male SR-04 Header, J5 USB_B_Micro, J6 3 Pin Male Servo Header, J7 3 Pin Male Servo Header, J8 3 Pin Male Servo Header, J9 3 Pin Male Servo Header, Q1 SMD-MOSFET-P-CH-20V-2A-FDN340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, SW1 SMD Button, SW2 SMD Button, SW3 SMD Button, SW4 SMD Button, U1 L7805CDT-TR, U2 DRV8833PW, U3 ATmega2560-16AU, U4 CP2102N-A01-GQFN24, Y1 16MHz Resonator

Commit message: V1.1
Parts:
- added IC1: APA102, ZigerBot:APA102-2020, F.Cu at (258.1, 103.3)
- added IC10: APA102, ZigerBot:APA102-2020, F.Cu at (270.9, 106.6)
- added IC11: APA102, ZigerBot:APA102-2020, F.Cu at (258.1, 109.9)
- added IC12: APA102, ZigerBot:APA102-2020, F.Cu at (261.2, 109.9)
- added IC13: APA102, ZigerBot:APA102-2020, F.Cu at (264.4, 109.9)
- added IC14: APA102, ZigerBot:APA102-2020, F.Cu at (267.6, 109.9)
- added IC15: APA102, ZigerBot:APA102-2020, F.Cu at (270.9, 109.9)
- added IC16: APA102, ZigerBot:APA102-2020, F.Cu at (258.1, 113.2)
- added IC17: APA102, ZigerBot:APA102-2020, F.Cu at (261.2, 113.2)
- added IC18: APA102, ZigerBot:APA102-2020, F.Cu at (264.4, 113.2)
- added IC19: APA102, ZigerBot:APA102-2020, F.Cu at (267.6, 113.2)
- added IC2: APA102, ZigerBot:APA102-2020, F.Cu at (261.2, 103.3)
- added IC20: APA102, ZigerBot:APA102-2020, F.Cu at (270.9, 113.2)
- added IC21: APA102, ZigerBot:APA102-2020, F.Cu at (258.1, 116.5)
- added IC22: APA102, ZigerBot:APA102-2020, F.Cu at (261.2, 116.5)
- added IC23: APA102, ZigerBot:APA102-2020, F.Cu at (264.4, 116.5)
- added IC24: APA102, ZigerBot:APA102-2020, F.Cu at (267.6, 116.5)
- added IC25: APA102, ZigerBot:APA102-2020, F.Cu at (270.9, 116.5)
- added IC3: APA102, ZigerBot:APA102-2020, F.Cu at (264.4, 103.3)
- added IC4: APA102, ZigerBot:APA102-2020, F.Cu at (267.6, 103.3)
- added IC5: APA102, ZigerBot:APA102-2020, F.Cu at (270.9, 103.3)
- added IC6: APA102, ZigerBot:APA102-2020, F.Cu at (258.1, 106.6)
- added IC7: APA102, ZigerBot:APA102-2020, F.Cu at (261.2, 106.6)
- added IC8: APA102, ZigerBot:APA102-2020, F.Cu at (264.4, 106.6)
- added IC9: APA102, ZigerBot:APA102-2020, F.Cu at (267.6, 106.6)
- C1, C10, C11, C12, C13, C14, C15, C16, C17, C18, C19, C2, C20, C21, C22, C23, C24, C25, C26, C27, C28, C29, C3, C30, C31, C32, C33, C34, C35, C36, C37, C38, C39, C4, C5, C6, C7, C8, C9: footprint Capacitors_SMD:C_0402 -> Capacitors_SMD:C_0805
- R1, R10, R12, R2, R3, R4, R5, R6, R7, R8, R9: footprint Resistors_SMD:R_0402 -> Resistors_SMD:R_0805
- U2: value DRV8833PW -> DRV8833PWPR; footprint Housings_SSOP:TSSOP-16-1EP_4.4x5mm_Pitch0.65mm -> digikey-footprints:TSSOP-16-1EP_W4.40mm
Connections:
- net /MotInA renamed /AOUT2
- net /MotInB renamed /BOUT2
- net /MotOutA renamed /AOUT1
- net /MotOutB renamed /BOUT1
- C2 pad 1: Net-(C2-Pad1) -> GND
- C3 pad 2: Net-(C2-Pad1) -> GND
- C5 pad 2: Net-(C2-Pad1) -> GND
- C6 pad 2: Net-(C2-Pad1) -> GND
- Q1 pad 1: Net-(C2-Pad1) -> GND
- R7 pad 2: Net-(C2-Pad1) -> GND
- R8 pad 2: Net-(C2-Pad1) -> GND
- U1 pad 2: Net-(C2-Pad1) -> GND
- U2 pad 13: Net-(C2-Pad1) -> GND
- U2 pad 17: (no net) -> GND
Routing:
- net GND: track 399.5 -> 559.8 mm, vias 45 -> 71
- net 5V: track 292.0 -> 432.7 mm, vias 0 -> 26
- net Net-(IC5-Pad3): track 0.00 -> 54.2 mm
- net Net-(IC5-Pad2): track 0.00 -> 51.4 mm
- net Net-(IC10-Pad3): track 0.00 -> 45.1 mm
- net Net-(IC10-Pad2): track 0.00 -> 42.3 mm
- net Net-(IC15-Pad3): track 0.00 -> 35.9 mm
- net Net-(IC15-Pad2): track 0.00 -> 33.2 mm
- net Net-(IC20-Pad3): track 0.00 -> 27.0 mm
- net Net-(IC20-Pad2): track 0.00 -> 24.1 mm
- net Net-(IC8-Pad3): track 0.00 -> 1.50 mm
- net Net-(IC8-Pad2): track 0.00 -> 1.50 mm
- net Net-(IC7-Pad3): track 0.00 -> 1.50 mm
- net Net-(IC7-Pad2): track 0.00 -> 1.50 mm
- net Net-(IC6-Pad3): track 0.00 -> 1.50 mm
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Other:
- copper layers 2 -> 4
- net class Default: clearance 0.2 -> 0.1524; trace_width 0.25 -> 0.1524
- net class Power: trace_width 0.8 -> 0.2
- net class Signal: clearance 0.2 -> 0.1524; trace_width 0.25 -> 0.1524
- rule trace_clearance: 0.2 -> 0.1524
- rule trace_min: 0.2 -> 0.1524
- rule via_min_size: 0.4 -> 0.3
- board text added: "0"
- board text added: "10"
- board text added: "14"
- board text added: "15"
- board text added: "19"
- board text added: "20"
- board text added: "24"
- board text added: "4"
- board text added: "5"
- board text added: "9"
