File: Hardware/pcb/ZigerBot/ZigerBot.sch (KiCad schematic (older format))
At the start: 34 parts, among them J1 Screw_Terminal_01x03, J2 Screw_Terminal_01x02, J3 Screw_Terminal_01x02, U1 L7805, U2 NXP 74HC04, U3 L298P

Commit message: PCB erweitert
Parts:
- removed D1: LED Blue, LEDs:LED_1206_HandSoldering, symbol Device:LED
- removed D10, D11, D12, D3, D4, D5, D6, D9: SR140, ZigerBot:D_DO-41_SOD81_P10.16mm_Horizontal, symbol Device:D_Schottky
- removed D13, D15, D7, D8: LED Red, LEDs:LED_1206_HandSoldering, symbol Device:LED
- removed D14: LED BLUE, LEDs:LED_1206_HandSoldering, symbol Device:LED
- removed D16, D2: LED Yellow, LEDs:LED_1206_HandSoldering, symbol Device:LED
- removed J1: Screw_Terminal_01x03, Connectors_Terminal_Blocks:TerminalBlock_bornier-3_P5.08mm, symbol Connector:Screw_Terminal_01x03
- removed J2, J3: Screw_Terminal_01x02, Connectors_Terminal_Blocks:TerminalBlock_bornier-2_P5.08mm, symbol Connector:Screw_Terminal_01x02
- removed JP1: Jumper, Pin_Headers:Pin_Header_Straight_1x02_Pitch2.54mm, symbol Device:Jumper
- removed R1, R2, R3, R4, R5, R6, R7, R8: 1k, Resistors_SMD:R_1206_HandSoldering, symbol Device:R
- removed U3: L298P, Housings_SOIC:HSOP-20-1EP_11.0x15.9mm_Pitch1.27mm_SlugDown, symbol Driver_Motor:L298P
- removed XA1: Arduino_Uno_Shield, Arduino:Arduino_Uno_Shield, symbol arduino:Arduino_Uno_Shield
- added C10, C11, C12, C4, C5, C8, C9: 0.1uF, Capacitor_SMD:C_0805_2012Metric, symbol Device:C
- added C3, C6: 4.7uF, Capacitor_SMD:C_0805_2012Metric, symbol Device:C
- added C7: 0.33uF, Capacitor_SMD:C_0805_2012Metric, symbol Device:C
- added D1, D19, D2, D7, D8: SMD LED red, SeeedOPL-LED:LED-0805, symbol SeeedOPL-LED:SMD-LED-CLEAR-RED_0805_
- added D10, D11, D12, D3, D4, D5, D6, D9: SCHOTTKY-40V-1A, SeeedOPL-Diode:DO-214AC, symbol SeeedOPL-Diode:SMD-DIODE-SCHOTTKY-40V-1A_DO-214AC_
- added D13, D15: SMD LED blue, SeeedOPL-LED:LED-0805, symbol SeeedOPL-LED:SMD-LED-CLEAR-BLUE_0805_
- added D14, D16, D20: SMD LED yellow, SeeedOPL-LED:LED-0805, symbol SeeedOPL-LED:SMD-LED-CLEAR-YELLOW_0805_
- added D17: SP0503BAHT, Package_TO_SOT_SMD:SOT-143, symbol Power_Protection:SP0503BAHT
- added D18: Schottky SS54B, SeeedOPL-Diode:DO-214AA, symbol SeeedOPL-Diode:SMD-DIODE-SCHOTTKY-28V-5A_DO-214AA_
- added J1: Power, SeeedOPL-Connector:H3-5.0-15.5X8.0MM, symbol SeeedOPL-Connector:SCREW-TERMINAL-GREEN_3P-5.0_
- added J2: Motor A, SeeedOPL-Connector:H2-5.0-10.5X8.0MM, symbol SeeedOPL-Connector:SCREW-TERMINAL-GREEN_2P-5.0_
- added J3: Motor B, SeeedOPL-Connector:H2-5.0-10.5X8.0MM, symbol SeeedOPL-Connector:SCREW-TERMINAL-GREEN_2P-5.0_
- added J4: Jumper, SeeedOPL-Connector:H2-2.54, symbol SeeedOPL-Connector:DIP-BLACK-MALE-HEADER-VERT_2P-2.54_
- added J5: USB_B_Micro, Connector_USB:USB_Micro-B_Amphenol_10103594-0001LF_Horizontal, symbol Connector:USB_B_Micro
- added R1, R2, R3, R4, R5, R6, R7, R8, R9: 1k, Resistor_SMD:R_0805_2012Metric, symbol SeeedOPL-Resistor:SMD-RES-1K-5%-1_8W_0805_
- added R10, R11, R12: 10k, Resistor_SMD:R_0805_2012Metric, symbol SeeedOPL-Resistor:SMD-RES-1K-5%-1_8W_0805_
- added U3: L298P, SeeedOPL-IC:SOIC20G-1.27-16X11MM, symbol SeeedOPL-IC:DRIVER-L298P_SOIC20_
- added U4: ATMEGA2560-16AU, SeeedOPL-IC:TQFP100-0.5-14X14MM, symbol SeeedOPL-IC:MCU-ATMEGA2560-16AU_TQFP100_
- added U5: CP2102N-A01-GQFN24, Package_DFN_QFN:QFN-24-1EP_4x4mm_P0.5mm_EP2.6x2.6mm, symbol Interface_USB:CP2102N-A01-GQFN24
- added Y1: C16M000000S004, symbol Device:Resonator
- C1, C2: value 0.1uF C1206S104M5RACTU -> 0.1uF; footprint Capacitors_SMD:C_1206_HandSoldering -> Capacitor_SMD:C_0805_2012Metric
- U1: value L7805 -> L7805CV; footprint Power_Integrations:TO-220 -> Package_TO_SOT_SMD:TO-252-2; MPN (none) -> L7805CV; SKU (none) -> 310030010
- U2: footprint Housings_SOIC:SOIC-14_3.9x8.7mm_Pitch1.27mm -> Package_SO:SOIC-14_3.9x8.7mm_P1.27mm
- U2: footprint Housings_SOIC:SOIC-14_3.9x8.7mm_Pitch1.27mm -> Package_SO:SOIC-14_3.9x8.7mm_P1.27mm; MPN (none) -> 74HCU04D
Connections:
- net labels added: DTRmega, DirMotA, DirMotB, EnaMotA, EnaMotB, RXmega, TXmega
- net labels removed: 3.3V, A0, A1, A2, A3, A4, A5, AREF, D0, D1, D10, D11, D12, D2, D3, D4, D5, D6, D7, D8, D9, IOREF, RST, SCL, SDA
- wire segments 160 -> 248
- no-connect marks 0 -> 5
Other:
- note removed: "27.09.2018"
- note removed: "LED Widerstände 1k\n"
- note removed: "VS 0.1µF 50V 20% Ceramic Capacitor\nVSS 47µF 35V 20% Radial Aluminum Capacitor\n1N4001 or 1A/40V/500mV"
- note removed: "ZigerBot"

Commit message: Added all peripheral components
Parts:
- removed C1, C4: 0.1uF, Capacitor_SMD:C_0805_2012Metric, symbol Device:C
- removed D1, D2, D7, D8: SMD LED red, SeeedOPL-LED:LED-0805, symbol SeeedOPL-LED:SMD-LED-CLEAR-RED_0805_
- removed D10, D11, D12, D3, D4, D5, D6, D9: SCHOTTKY-40V-1A, SeeedOPL-Diode:DO-214AC, symbol SeeedOPL-Diode:SMD-DIODE-SCHOTTKY-40V-1A_DO-214AC_
- removed D18: Schottky SS54B, SeeedOPL-Diode:DO-214AA, symbol SeeedOPL-Diode:SMD-DIODE-SCHOTTKY-28V-5A_DO-214AA_
- removed J1: Power, SeeedOPL-Connector:H3-5.0-15.5X8.0MM, symbol SeeedOPL-Connector:SCREW-TERMINAL-GREEN_3P-5.0_
- removed J4: Jumper, SeeedOPL-Connector:H2-2.54, symbol SeeedOPL-Connector:DIP-BLACK-MALE-HEADER-VERT_2P-2.54_
- removed R1, R2, R3, R4: 1k, Resistor_SMD:R_0805_2012Metric, symbol SeeedOPL-Resistor:SMD-RES-1K-5%-1_8W_0805_
- removed U2: NXP 74HC04, Package_SO:SOIC-14_3.9x8.7mm_P1.27mm, symbol 74xx:74HC04
- removed U3: L298P, SeeedOPL-IC:SOIC20G-1.27-16X11MM, symbol SeeedOPL-IC:DRIVER-L298P_SOIC20_
- added BZ?: Buzzer CEM-1203(42), symbol Device:Buzzer
- added C? (x3): 10uF 16V, symbol Device:C_Small
- added C?: 0.1 uF, symbol Device:C_Small
- added C? (x25): 100nF, symbol Device:C_Small
- added CN? (x4): 3 Pin Male Servo Header, symbol SeeedOPL-Connector:DIP-BLACK-MALE-HEADER-VERT_3P-2.54_
- added D?: SMD LED green FAULT, SeeedOPL-LED:LED-0805, symbol SeeedOPL-LED:SMD-LED-CLEAR-RED_0805_
- added D? (x25): WS2812B, LED_SMD:LED_WS2812B_PLCC4_5.0x5.0mm_P3.2mm, symbol LED:WS2812B
- added J?: M Power, SeeedOPL-Connector:H2-5.0-10.5X8.0MM, symbol SeeedOPL-Connector:SCREW-TERMINAL-GREEN_2P-5.0_
- added J?: 4 Pin Male SR-04 Header, symbol SeeedOPL-Connector:DIP-BLACK-MALE-HEADER-VERT_4P-2.54_
- added JP?: Jumper, symbol Device:Jumper_NC_Dual
- added Q?: SMD-MOSFET-P-CH-20V-2A-FDN340P_SOT-23_, symbol SeeedOPL-Transistor:SMD-MOSFET-P-CH-20V-2A-FDN340P_SOT-23_
- added R? (x2): 0.2 Ohm, symbol Device:R_Small
- added R?: 10k, Resistor_SMD:R_0805_2012Metric, symbol SeeedOPL-Resistor:SMD-RES-1K-5%-1_8W_0805_
- added R?: 100 Ohm, symbol SeeedOPL-Resistor:SMD-RES-100R-5%-1_8W_0805_
- added RV? (x2): Potentiometer, symbol Device:R_POT
- added SW? (x4): SMD Button, symbol SeeedOPL-Switch:SMD-BUTTON_4P-5.2X5.2X1.5MM-SKQGADE010_
- added U?: DRV8833PW, Package_SO:TSSOP-16_4.4x5mm_P0.65mm, symbol Driver_Motor:DRV8833PW
Connections:
- net labels added: 5V, AIN1, AIN2, BIN1, BIN2, Button1, Button2, Button3, Button4, Buzz, Echo, Pot1, Pot2, Servo1, Servo2, Servo3, Servo4, Trig, VCP
- net labels removed: DirMotA, DirMotB, EnaMotA, EnaMotB, VS, VSS
- wire segments 248 -> 298
- no-connect marks 5 -> 2
Other:
- note added: "2.7-10.8V"
- note added: "Atmega2560"
- note added: "Buttons"
- note added: "Motor Driver and Motor Power"
- note added: "Potentiometer"
- note added: "Range sensor connector"
- note added: "Servo-Connectors"
- note added: "Speaker"
- note added: "USB to UART Bridge"
- note added: "WS2812B LED Matrix"
- moved on the sheet: C10, C11, C12, C2, C3, C5, C6, C7, C8, C9, J2, J3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

Commit message: PCB changed
Parts:
- removed CN? (x4): 3 Pin Male Servo Header, symbol SeeedOPL-Connector:DIP-BLACK-MALE-HEADER-VERT_3P-2.54_
- removed D14, D16: SMD LED yellow, SeeedOPL-LED:LED-0805, symbol SeeedOPL-LED:SMD-LED-CLEAR-YELLOW_0805_
- removed D15: SMD LED blue, SeeedOPL-LED:LED-0805, symbol SeeedOPL-LED:SMD-LED-CLEAR-BLUE_0805_
- removed SW? (x3): SMD Button, symbol SeeedOPL-Switch:SMD-BUTTON_4P-5.2X5.2X1.5MM-SKQGADE010_
- removed U4: ATMEGA2560-16AU, SeeedOPL-IC:TQFP100-0.5-14X14MM, symbol SeeedOPL-IC:MCU-ATMEGA2560-16AU_TQFP100_
- removed Y1: C16M000000S004, symbol Device:Resonator
- added D3, D7: SMD LED yellow, ZigerBot:LED_0603, symbol Device:LED
- added D6: SMD LED blue, ZigerBot:LED_0603, symbol Device:LED
- added J6, J7, J8, J9: 3 Pin Male Servo Header, Pin_Headers:Pin_Header_Straight_1x03_Pitch2.54mm, symbol Connector:Conn_01x03_Female
- added SW2, SW3, SW4: SMD Button, Buttons_Switches_SMD:SW_SPST_SKQG, symbol Switch:SW_SPST
- added U3: ATmega2560-16AU, Package_QFP:TQFP-100_14x14mm_P0.5mm, symbol MCU_Microchip_ATmega:ATmega2560-16AU
- added Y1: 16MHz Resonator, ZigerBot:Resonator_SMD_muRata_CSTNE16M0V530000_3pin_3.2x1.3x0.9mm, symbol Device:Resonator_Small
- BZ1: renamed from BZ?; footprint (none) -> ZigerBot:BUZZER_CEM-1203(24)_12mm_6.5mm_0.6mm
- C1: renamed from C9; footprint Capacitor_SMD:C_0805_2012Metric -> Capacitors_SMD:C_0402
- C10: renamed from C12; footprint Capacitor_SMD:C_0805_2012Metric -> Capacitors_SMD:C_0402
- C11, C12, C13, C14, C15, C16, C17, C18, C19, C20, C23, C24, C25, C26, C27, C28, C29, C30, C31, C32, C35, C36, C37, C38, C39, C4, C5, C6, C7: renamed from C?; footprint (none) -> Capacitors_SMD:C_0402
- C2: renamed from C7; footprint Capacitor_SMD:C_0805_2012Metric -> Capacitors_SMD:C_0402
- C21: renamed from C5; footprint Capacitor_SMD:C_0805_2012Metric -> Capacitors_SMD:C_0402
- C22: renamed from C6; footprint Capacitor_SMD:C_0805_2012Metric -> Capacitors_SMD:C_0402
- C3: renamed from C8; footprint Capacitor_SMD:C_0805_2012Metric -> Capacitors_SMD:C_0402
- C33: renamed from C2; footprint Capacitor_SMD:C_0805_2012Metric -> Capacitors_SMD:C_0402
- C34: renamed from C3; footprint Capacitor_SMD:C_0805_2012Metric -> Capacitors_SMD:C_0402
- C8: renamed from C10; footprint Capacitor_SMD:C_0805_2012Metric -> Capacitors_SMD:C_0402
- C9: renamed from C11; footprint Capacitor_SMD:C_0805_2012Metric -> Capacitors_SMD:C_0402
- D1: renamed from D19; footprint SeeedOPL-LED:LED-0805 -> ZigerBot:LED_0603
- D10, D11, D12, D13, D14, D15, D16, D17, D18, D19, D20, D21, D22, D24, D25, D26, D27, D28, D29, D30, D31, D32, D33, D8, D9: renamed from D?; footprint LED_SMD:LED_WS2812B_PLCC4_5.0x5.0mm_P3.2mm -> ZigerBot:LED_WS2812B-PLCC4
- D2: renamed from D13; footprint SeeedOPL-LED:LED-0805 -> ZigerBot:LED_0603; symbol SeeedOPL-LED:SMD-LED-CLEAR-BLUE_0805_ -> Device:LED; MPN 17-215SURC_S530-A2_TR8 -> (none); SKU 304090046 -> (none)
- D4: renamed from D20; footprint SeeedOPL-LED:LED-0805 -> ZigerBot:LED_0603
- D5: renamed from D?; footprint SeeedOPL-LED:LED-0805 -> ZigerBot:LED_0603
- J4: renamed from J?; footprint (none) -> SeeedOPL-Connector:H4-2.54
- JP1: renamed from JP?; footprint (none) -> Pin_Headers:Pin_Header_Straight_1x03_Pitch2.54mm
- Q1: renamed from Q?; footprint (none) -> TO_SOT_Packages_SMD:SOT-23
- R1, R7, R8: renamed from R?; footprint (none) -> Resistors_SMD:R_0402
- R10: renamed from R7; footprint Resistor_SMD:R_0805_2012Metric -> Resistors_SMD:R_0402
- R11: renamed from R8; footprint Resistor_SMD:R_0805_2012Metric -> Resistors_SMD:R_0402
- R12: renamed from R9; footprint Resistor_SMD:R_0805_2012Metric -> Resistors_SMD:R_0402
- R2: renamed from R10; footprint Resistor_SMD:R_0805_2012Metric -> Resistors_SMD:R_0402
- R3: renamed from R11; footprint Resistor_SMD:R_0805_2012Metric -> Resistors_SMD:R_0402
- R4: renamed from R5; footprint Resistor_SMD:R_0805_2012Metric -> Resistors_SMD:R_0402
- R5: renamed from R6; footprint Resistor_SMD:R_0805_2012Metric -> Resistors_SMD:R_0402
- R6: renamed from R12; footprint Resistor_SMD:R_0805_2012Metric -> Resistors_SMD:R_0402
- R9: renamed from R?; footprint Resistor_SMD:R_0805_2012Metric -> Resistors_SMD:R_0402
- RV1, RV2: renamed from RV?; footprint (none) -> Potentiometers:Potentiometer_Trimmer-EVM3E
- SW1: renamed from SW?; footprint (none) -> Buttons_Switches_SMD:SW_SPST_SKQG; symbol SeeedOPL-Switch:SMD-BUTTON_4P-5.2X5.2X1.5MM-SKQGADE010_ -> Switch:SW_SPST
- U4: renamed from U5; footprint Package_DFN_QFN:QFN-24-1EP_4x4mm_P0.5mm_EP2.6x2.6mm -> Housings_DFN_QFN:QFN-24-1EP_4x4mm_Pitch0.5mm
- gave numbers to parts that had none: 2
- renumbered D17 to D23, J2 to J1
Connections:
- wire segments 298 -> 283
Other:
- note added: "Cap between Pin 99 and 100"
- note added: "Caps between Pins 31/32 and 61/62"
- moved on the sheet: C1, C10, C8, C9, R3, R6

Commit message: Updated Package Info
Parts:
- D1, D5: symbol SeeedOPL-LED:SMD-LED-CLEAR-RED_0805_ -> Device:LED; MPN 17-215SURC_S530-A2_TR8 -> (none); SKU 304090046 -> (none)
- D23: footprint Package_TO_SOT_SMD:SOT-143 -> TO_SOT_Packages_SMD:SOT-143_Handsoldering
- D4: symbol SeeedOPL-LED:SMD-LED-CLEAR-YELLOW_0805_ -> Device:LED; MPN 17-215SURC_S530-A2_TR8 -> (none); SKU 304090046 -> (none)
- J5: footprint Connector_USB:USB_Micro-B_Amphenol_10103594-0001LF_Horizontal -> Connectors_USB:USB_Micro-B_Molex-105017-0001
- U1: value L7805CV -> L7805CDT-TR; footprint Package_TO_SOT_SMD:TO-252-2 -> TO_SOT_Packages_SMD:TO-252-2; MPN L7805CV -> L7805CDT-TR
- U2: footprint Package_SO:TSSOP-16_4.4x5mm_P0.65mm -> Housings_SSOP:TSSOP-16-1EP_4.4x5mm_Pitch0.65mm
- U3: footprint Package_QFP:TQFP-100_14x14mm_P0.5mm -> Housings_QFP:TQFP-100_14x14mm_Pitch0.5mm
Changed lines of the file:
@@
 P 2600 1100
 F 0 "U1" H 2600 1350 45  0000 C CNN
-F 1 "L7805CV" H 2600 1250 45  0000 C CNN
-F 2 "Package_TO_SOT_SMD:TO-252-2" H 2600 1100 50  0001 C CNN
+F 1 "L7805CDT-TR" H 2600 1250 45  0000 C CNN
+F 2 "TO_SOT_Packages_SMD:TO-252-2" H 2600 1100 50  0001 C CNN
 F 3 "" H 2600 1100 50  0001 C CNN
-F 4 "L7805CV" H 2630 1250 20  0001 C CNN "MPN"
+F 4 "L7805CDT-TR" H 2630 1250 20  0001 C CNN "MPN"
 F 5 "310030010" H 2630 1250 20  0001 C CNN "SKU"
 	1    2600 1100
@@
 F 0 "J5" H 1055 7167 50  0000 C CNN
 F 1 "USB_B_Micro" H 1055 7076 50  0000 C CNN
-F 2 "Connector_USB:USB_Micro-B_Amphenol_10103594-0001LF_Horizontal" H 1150 6650 50  0001 C CNN
+F 2 "Connectors_USB:USB_Micro-B_Molex-105017-0001" H 1150 6650 50  0001 C CNN
 F 3 "~" H 1150 6650 50  0001 C CNN
 F 4 "10118193-0001LF" H 1000 6700 50  0001 C CNN "MPN"
@@
 $EndComp
 $Comp
-L SeeedOPL-LED:SMD-LED-CLEAR-YELLOW_0805_ D4
+L Device:LED D4
 U 1 1 5BDAE84A
 P 10600 3700
@@
 F 2 "ZigerBot:LED_0603" H 10600 3700 50  0001 C CNN
 F 3 "" H 10600 3700 50  0001 C CNN
-F 4 "17-215SURC_S530-A2_TR8" H 10630 3850 20  0001 C CNN "MPN"
-F 5 "304090046" H 10630 3850 20  0001 C CNN "SKU"
 	1    10600 3700
-	1    0    0    -1
+	-1   0    0    1
 $EndComp
 Text Label 10750 3700 0    50   ~ 0
@@
 Connection ~ 2900 1100
 $Comp
-L SeeedOPL-LED:SMD-LED-CLEAR-RED_0805_ D1
+L Device:LED D1
 U 1 1 5BDAEEEA
 P 3350 1100
-F 0 "D1" H 3350 1429 45  0000 C CNN
-F 1 "SMD LED red" H 3350 1345 45  0000 C CNN
+F 0 "D1" H 3350 1000 45  0000 C CNN
+F 1 "SMD LED red" H 3300 900 45  0000 C CNN
 F 2 "ZigerBot:LED_0603" H 3350 1100 50  0001 C CNN
 F 3 "" H 3350 1100 50  0001 C CNN
-F 4 "17-215SURC_S530-A2_TR8" H 3380 1250 20  0001 C CNN "MPN"
-F 5 "304090046" H 3380 1250 20  0001 C CNN "SKU"
 	1    3350 1100
-	1    0    0    -1
+	-1   0    0    1
 $EndComp
 Text GLabel 3500 1100 2    50   Input ~ 0
@@
 F 0 "D23" H 2005 7146 50  0000 L CNN
 F 1 "SP0503BAHT" H 2005 7055 50  0000 L CNN
-F 2 "Package_TO_SOT_SMD:SOT-143" H 2025 7050 50  0001 L CNN
+F 2 "TO_SOT_Packages_SMD:SOT-143_Handsoldering" H 2025 7050 50  0001 L CNN
 F 3 "http://www.littelfuse.com/~/media/files/littelfuse/technical%20resources/documents/data%20sheets/sp05xxba.pdf" H 1925 7225 50  0001 C CNN
 	1    1800 7100
@@
 F 0 "U2" H 3850 2064 50  0000 C CNN
 F 1 "DRV8833PW" H 3850 1973 50  0000 C CNN
-F 2 "Package_SO:TSSOP-16_4.4x5mm_P0.65mm" H 4300 3300 50  0001 L CNN
+F 2 "Housings_SSOP:TSSOP-16-1EP_4.4x5mm_Pitch0.65mm" H 4300 3300 50  0001 L CNN
 F 3 "http://www.ti.com/lit/ds/symlink/drv8833.pdf" H 3700 3400 50  0001 C CNN
 	1    3850 2850
@@
 $EndComp
 $Comp
-L SeeedOPL-LED:SMD-LED-CLEAR-RED_0805_ D5
+L Device:LED D5
 U 1 1 5BE29165
 P 4900 2750
-F 0 "D5" H 4900 3079 45  0000 C CNN
-F 1 "SMD LED green FAULT" H 4900 2995 45  0000 C CNN
+F 0 "D5" H 4900 2650 45  0000 C CNN
+F 1 "SMD LED green FAULT" H 4800 2500 45  0000 C CNN
 F 2 "ZigerBot:LED_0603" H 4900 2750 50  0001 C CNN
 F 3 "" H 4900 2750 50  0001 C CNN
-F 4 "17-215SURC_S530-A2_TR8" H 4930 2900 20  0001 C CNN "MPN"
-F 5 "304090046" H 4930 2900 20  0001 C CNN "SKU"
 	1    4900 2750
-	1    0    0    -1
+	-1   0    0    1
 $EndComp
 Text GLabel 5050 2750 2    50   Input ~ 0
@@
 F 0 "U3" H 9350 1714 50  0000 C CNN
 F 1 "ATmega2560-16AU" H 9350 1623 50  0000 C CNN
-F 2 "Package_QFP:TQFP-100_14x14mm_P0.5mm" H 9350 4700 50  0001 C CIN
+F 2 "Housings_QFP:TQFP-100_14x14mm_Pitch0.5mm" H 9350 4700 50  0001 C CIN
 F 3 "http://ww1.microchip.com/downloads/en/DeviceDoc/Atmel-2549-8-bit-AVR-Microcontroller-ATmega640-1280-1281-2560-2561_datasheet.pdf" H 9350 4700 50  0001 C CNN
 	1    9350 4700
