File: Hardware/pcb/ZigerBot/ZigerBot.sch (KiCad schematic (older format))
At the start: 105 parts, among them J1 Motor A, J10 ICSP, J2 M Power, J3 Motor B, J4 4 Pin Male SR-04 Header, J5 USB_B_Micro, J6 3 Pin Male Servo Header, J7 3 Pin Male Servo Header, J8 3 Pin Male Servo Header, J9 3 Pin Male Servo Header, Q1 SMD-MOSFET-P-CH-20V-2A-FDN340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, SW1 SMD Button, SW2 SMD Button, SW3 SMD Button, SW4 SMD Button, U1 L7805CDT-TR, U2 DRV8833PW, U3 ATmega2560-16AU, U4 CP2102N-A01-GQFN24, Y1 16MHz Resonator

Commit message: V1.1
Parts:
- removed U2: DRV8833PW, Housings_SSOP:TSSOP-16-1EP_4.4x5mm_Pitch0.65mm, symbol Driver_Motor:DRV8833PW
- added IC1, IC10, IC11, IC12, IC13, IC14, IC15, IC16, IC17, IC18, IC19, IC2, IC20, IC21, IC22, IC23, IC24, IC25, IC3, IC4, IC5, IC6, IC7, IC8, IC9: APA102, ZigerBot:APA102-2020, symbol ZigerBot-rescue:APA102
- added U2: DRV8833PWPR, digikey-footprints:TSSOP-16-1EP_W4.40mm, symbol dk_PMIC-Full-Half-Bridge-Drivers:DRV8833PWPR
- BZ1: Digi-Key_PN (none) -> 102-1153-ND
- C1, C10, C11, C12, C13, C14, C15, C16, C17, C18, C19, C20, C21, C23, C24, C25, C26, C27, C28, C29, C3, C30, C31, C32, C33, C35, C36, C37, C38, C39, C4, C8, C9: footprint Capacitors_SMD:C_0402 -> Capacitors_SMD:C_0805; Digi-Key_PN (none) -> 311-1141-1-ND
- C2: footprint Capacitors_SMD:C_0402 -> Capacitors_SMD:C_0805; Digi-Key_PN (none) -> 311-3385-1-ND
- C22, C34: footprint Capacitors_SMD:C_0402 -> Capacitors_SMD:C_0805; Digi-Key_PN (none) -> 311-1863-1-ND
- C5, C6, C7: footprint Capacitors_SMD:C_0402 -> Capacitors_SMD:C_0805; Digi-Key_PN (none) -> 490-3886-1-ND
- D1: Digi-Key_PN (none) -> 160-1436-1-ND
- D10, D11, D12, D13, D14, D15, D16, D17, D18, D19, D20, D21, D22, D24, D25, D26, D27, D28, D29, D30, D31, D32, D33, D8, D9: Digi-Key_PN (none) -> 1528-1104-ND
- D2, D3: Digi-Key_PN (none) -> 160-1038-ND
- D23: symbol Power_Protection:SP0503BAHT -> ZigerBot-rescue:SP0503BAHT-Power_Protection; Digi-Key_PN (none) -> F2715CT-ND
- D4: Digi-Key_PN (none) -> 160-1437-1-ND
- D5: Digi-Key_PN (none) -> 160-1435-1-ND
- J1, J2, J3: Digi-Key_PN (none) -> ED2609-ND
- J10: Digi-Key_PN (none) -> 609-3218-ND
- J4: Digi-Key_PN (none) -> 732-5317-ND
- J5: Digi-Key_PN (none) -> 609-4616-1-ND; MPN 10118193-0001LF -> (none)
- J6, J7, J8, J9, JP1: Digi-Key_PN (none) -> 732-5316-ND
- Q1: Digi-Key_PN (none) -> FDN340PCT-ND
- R1: footprint Resistors_SMD:R_0402 -> Resistors_SMD:R_0805; Digi-Key_PN (none) -> 311-100CRCT-ND; MPN RC0805JR-07100RL -> (none)
- R10, R12, R4: footprint Resistors_SMD:R_0402 -> Resistors_SMD:R_0805; Digi-Key_PN (none) -> 311-1.00KCRCT-ND; MPN RC0805JR-071KL -> (none)
- R2, R3, R6, R9: footprint Resistors_SMD:R_0402 -> Resistors_SMD:R_0805; Digi-Key_PN (none) -> 311-10.0KCRCT-ND; MPN RC0805JR-071KL -> (none)
- R5: footprint Resistors_SMD:R_0402 -> Resistors_SMD:R_0805; Digi-Key_PN (none) -> 311-470CRCT-ND; MPN RC0805JR-07100RL -> (none)
- R7, R8: footprint Resistors_SMD:R_0402 -> Resistors_SMD:R_0805; Digi-Key_PN (none) -> 311-.20SCT-ND
- RV1, RV2: Digi-Key_PN (none) -> 1528-1997-ND
- SW1, SW2, SW3, SW4: Digi-Key_PN (none) -> CKN9087CT-ND; MPN SKQGADE010 -> PTS645SK50SMTR92 LFS
- U1: Digi-Key_PN (none) -> 497-7255-1-ND
- U3: symbol MCU_Microchip_ATmega:ATmega2560-16AU -> ZigerBot-rescue:ATmega2560-16AU-MCU_Microchip_ATmega; Digi-Key_PN (none) -> ATMEGA2560-16AU-ND
- U4: Digi-Key_PN (none) -> 336-4737-1-ND
- Y1: Digi-Key_PN (none) -> CSTNE16M0V53C000R0
Connections:
- net labels added: AOUT1, AOUT2, BOUT1, BOUT2
- net labels removed: MotInA, MotInB, MotOutA, MotOutB
- wire segments 270 -> 368
Other:
- moved on the sheet: C7, D5, R7, R8, R9
